File: intfield77.kicad_pcb (KiCad board)
At the start: 2 copper layers, 174 parts, among them J1 USB_C_Receptacle_USB2.0, SW1 RESET, SW2 BOOT, U1 STM32F072C8Tx, U2 SRV05-4, U3 XC6206PxxxMR

Commit message: Placed diodes and roughly placed other PCB components.
Parts:
- moved D77 498.8 mm to (393.7, 121.4), turned to 90 degrees
- moved D67 497.3 mm to (393.7, 102.4), turned to 90 degrees
- moved D34 480.5 mm to (388.9, 64.3), turned to 90 degrees
- moved D76 479.5 mm to (374.6, 121.4), turned to 90 degrees
- moved D50 478.7 mm to (381.8, 83.3), turned to 90 degrees
- moved D66 477.0 mm to (374.6, 102.4), turned to 90 degrees
- moved D17 472.2 mm to (384.2, 45.2), turned to 90 degrees
- moved D75 460.2 mm to (355.6, 121.4), turned to 90 degrees
- moved D33 458.8 mm to (365.1, 64.3), turned to 90 degrees
- moved D65 457.7 mm to (355.6, 102.4), turned to 90 degrees
- moved D49 447.7 mm to (350.8, 83.3), turned to 90 degrees
- moved D16 443.7 mm to (355.6, 45.2), turned to 90 degrees
- moved D32 439.5 mm to (346.1, 64.3), turned to 90 degrees
- moved D74 438.5 mm to (334.2, 121.4), turned to 90 degrees
- moved D64 438.3 mm to (336.6, 102.4), turned to 90 degrees
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Other:
- board outline added: 357.2 x 102.4 mm

Commit message: Shuffled MCU pins and realigned schema to 50 mils, but USB connector is not connected.
Parts:
- J1: footprint Type-C:HRO-TYPE-C-31-M-12-Assembly -> Type-C:HRO-TYPE-C-31-M-12
Connections:
- U1 pad 10: ROW14 -> ROW3
- U1 pad 11: ROW8 -> ROW4
- U1 pad 12: ROW7 -> ROW5
- U1 pad 14: ROW5 -> ROW7
- U1 pad 15: ROW4 -> ROW8
- U1 pad 16: ROW3 -> unconnected-(U1-PA6-Pad16)
- U1 pad 17: ROW2 -> unconnected-(U1-PA7-Pad17)
- U1 pad 18: ROW1 -> ROW14
- U1 pad 19: ROW0 -> ROW13
- U1 pad 2: unconnected-(U1-PC13-Pad2) -> ROW0
- U1 pad 20: COL3 -> ROW12
- U1 pad 21: COL4 -> ROW11
- U1 pad 22: COL5 -> ROW10
- U1 pad 25: COL6 -> unconnected-(U1-PB12-Pad25)
- U1 pad 26: COL7 -> COL2
- U1 pad 27: COL8 -> COL1
- U1 pad 28: COL9 -> COL0
- U1 pad 3: unconnected-(U1-PC14-Pad3) -> ROW1
- U1 pad 39: COL0 -> COL9
- U1 pad 4: unconnected-(U1-PC15-Pad4) -> ROW2
- U1 pad 40: COL1 -> COL8
- U1 pad 41: COL2 -> COL7
- U1 pad 42: ROW10 -> COL6
- U1 pad 43: ROW11 -> COL5
- U1 pad 45: ROW12 -> COL4
- U1 pad 46: ROW13 -> COL3

Commit message: Changed USB-C and reset button symbols and footprints, still problems.
Parts:
- J1: value USB_C_Receptacle_USB2.0 -> USB_C_Receptacle; footprint Type-C:HRO-TYPE-C-31-M-12 -> Connector_USB:USB_C_Receptacle_HRO_TYPE-C-31-M-12
- SW1: footprint random-keyboard-parts:SKQGADE010 -> Button_Switch_SMD:SW_Push_SPST_NO_Alps_SKRK
- moved C1 4.50 mm to (117.5, 80.0), turned to -90 degrees
- moved J1 3.37 mm to (107.2, 27.8)

Commit message: Fixed it, I think.
Parts:
- SW1: footprint Button_Switch_SMD:SW_Push_SPST_NO_Alps_SKRK -> Button_Switch_SMD:SW_SPST_SKQG_WithStem
- moved C7 1.59 mm to (108.0, 81.0)
- moved SW1 1.59 mm to (107.2, 100.0)
- moved J1 1.59 mm to (107.2, 29.4)
Changed lines of the file:
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@@
       (net 35 "Net-(D25-A)") (pinfunction "ROW") (pintype "passive"))
   )
-  (footprint "Button_Switch_SMD:SW_Push_SPST_NO_Alps_SKRK" (layer "F.Cu")
-    (at 107.15625 98.425 -90)
-    (descr "http://www.alps.com/prod/info/E/HTML/Tact/SurfaceMount/SKRK/SKRKAHE020.html")
-    (tags "SMD SMT button")
+  (footprint "Button_Switch_SMD:SW_SPST_SKQG_WithStem" (layer "F.Cu")
+    (at 107.15625 100.0125 -90)
+    (descr "ALPS 5.2mm Square Low-profile Type (Surface Mount) SKQG Series, With stem, http://www.alps.com/prod/info/E/HTML/Tact/SurfaceMount/SKQG/SKQGAFE010.html")
+    (tags "SPST Button Switch")
     (property "Sheetfile" "intfield77.kicad_sch")
     (property "Sheetname" "")
@@
     (property "ki_keywords" "switch normally-open pushbutton push-button")
     (attr smd)
-    (fp_text reference "SW1" (at 0 -2.25 -90) (layer "F.SilkS")
+    (fp_text reference "SW1" (at 0 -3.6 -90) (layer "F.SilkS")
         (effects (font (size 1 1) (thickness 0.15)))
     )
-    (fp_text value "RESET" (at 0 2.5 -90) (layer "F.Fab")
+    (fp_text value "RESET" (at 0 3.6 -90) (layer "F.Fab")
         (effects (font (size 1 1) (thickness 0.15)))
     )
+    (fp_text user "No F.Cu tracks" (at 2.5 0.2 -90) (layer "Cmts.User")
+        (effects (font (size 0.2 0.2) (thickness 0.03)))
+    )
+    (fp_text user "KEEP-OUT ZONE" (at -2.5 -0.2 -90) (layer "Cmts.User")
+        (effects (font (size 0.2 0.2) (thickness 0.03)))
+    )
+    (fp_text user "KEEP-OUT ZONE" (at 2.5 -0.2 -90) (layer "Cmts.User")
+        (effects (font (size 0.2 0.2) (thickness 0.03)))
+    )
+    (fp_text user "No F.Cu tracks" (at -2.5 0.2 -90) (layer "Cmts.User")
+        (effects (font (size 0.2 0.2) (thickness 0.03)))
+    )
     (fp_text user "${REFERENCE}" (at 0 0 -90) (layer "F.Fab")
-        (effects (font (size 1 1) (thickness 0.15)))
+        (effects (font (size 0.4 0.4) (thickness 0.06)))
     )
-    (fp_line (start -2.07 -1.57) (end 2.07 -1.57)
+    (fp_line (start -2.72 1.04) (end -2.72 -1.04)
+      (stroke (width 0.12) (type solid)) (layer "F.SilkS"))
+    (fp_line (start -1.45 -2.72) (end -1.94 -2.23)
       (stroke (width 0.12) (type solid)) (layer "F.SilkS"))
-    (fp_line (start -2.07 -1.27) (end -2.07 -1.57)
+    (fp_line (start -1.45 -2.72) (end 1.45 -2.72)
       (stroke (width 0.12) (type solid)) (layer "F.SilkS"))
-    (fp_line (start -2.07 1.57) (end -2.07 1.27)
+    (fp_line (start -1.45 2.72) (end -1.94 2.23)
       (stroke (width 0.12) (type solid)) (layer "F.SilkS"))
-    (fp_line (start 2.07 -1.57) (end 2.07 -1.27)
+    (fp_line (start -1.45 2.72) (end 1.45 2.72)
       (stroke (width 0.12) (type solid)) (layer "F.SilkS"))
-    (fp_line (start 2.07 1.27) (end 2.07 1.57)
+    (fp_line (start 1.45 -2.72) (end 1.94 -2.23)
       (stroke (width 0.12) (type solid)) (layer "F.SilkS"))
-    (fp_line (start 2.07 1.57) (end -2.07 1.57)
+    (fp_line (start 1.45 2.72) (end 1.94 2.23)
       (stroke (width 0.12) (type solid)) (layer "F.SilkS"))
-    (fp_line (start -2.75 -1.7) (end 2.75 -1.7)
+    (fp_line (start 2.72 1.04) (end 2.72 -1.04)
+      (stroke (width 0.12) (type solid)) (layer "F.SilkS"))
+    (fp_line (start -4.25 -2.85) (end -4.25 2.85)
       (stroke (width 0.05) (type solid)) (layer "F.CrtYd"))
-    (fp_line (start -2.75 1.7) (end -2.75 -1.7)
+    (fp_line (start -4.25 2.85) (end 4.25 2.85)
       (stroke (width 0.05) (type solid)) (layer "F.CrtYd"))
-    (fp_line (start 2.75 -1.7) (end 2.75 1.7)
+    (fp_line (start 4.25 -2.85) (end -4.25 -2.85)
       (stroke (width 0.05) (type solid)) (layer "F.CrtYd"))
-    (fp_line (start 2.75 1.7) (end -2.75 1.7)
+    (fp_line (start 4.25 2.85) (end 4.25 -2.85)
       (stroke (width 0.05) (type solid)) (layer "F.CrtYd"))
-    (fp_line (start -1.95 -1.45) (end 1.95 -1.45)
+    (fp_line (start -2.6 -1.4) (end -1.4 -2.6)
+      (stroke (width 0.1) (type solid)) (layer "F.Fab"))
+    (fp_line (start -2.6 1.4) (end -2.6 -1.4)
+      (stroke (width 0.1) (type solid)) (layer "F.Fab"))
+    (fp_line (start -1.865 0.95) (end -1.865 -0.95)
+      (stroke (width 0.1) (type solid)) (layer "F.Fab"))
+    (fp_line (start -1.4 -2.6) (end 1.4 -2.6)
+      (stroke (width 0.1) (type solid)) (layer "F.Fab"))
+    (fp_line (start -1.4 2.6) (end -2.6 1.4)
       (stroke (width 0.1) (type solid)) (layer "F.Fab"))
-    (fp_line (start -1.95 1.45) (end -1.95 -1.45)
+    (fp_line (start -0.95 -1.865) (end -1.865 -0.95)
       (stroke (width 0.1) (type solid)) (layer "F.Fab"))
-    (fp_line (start 1.95 -1.45) (end 1.95 1.45)
+    (fp_line (start -0.95 -1.865) (end 0.95 -1.865)
       (stroke (width 0.1) (type solid)) (layer "F.Fab"))
-    (fp_line (start 1.95 1.45) (end -1.95 1.45)
+    (fp_line (start -0.95 1.865) (end -1.865 0.95)
+      (stroke (width 0.1) (type solid)) (layer "F.Fab"))
+    (fp_line (start 0.95 -1.865) (end 1.865 -0.95)
+      (stroke (width 0.1) (type solid)) (layer "F.Fab"))
+    (fp_line (start 0.95 1.865) (end -0.95 1.865)
+      (stroke (width 0.1) (type solid)) (layer "F.Fab"))
+    (fp_line (start 0.95 1.865) (end 1.865 0.95)
+      (stroke (width 0.1) (type solid)) (layer "F.Fab"))
+    (fp_line (start 1.4 -2.6) (end 2.6 -1.4)
+      (stroke (width 0.1) (type solid)) (layer "F.Fab"))
+    (fp_line (start 1.4 2.6) (end -1.4 2.6)
+      (stroke (width 0.1) (type solid)) (layer "F.Fab"))
+    (fp_line (start 1.865 -0.95) (end 1.865 0.95)
+      (stroke (width 0.1) (type solid)) (layer "F.Fab"))
+    (fp_line (start 2.6 -1.4) (end 2.6 1.4)
+      (stroke (width 0.1) (type solid)) (layer "F.Fab"))
+    (fp_line (start 2.6 1.4) (end 1.4 2.6)
       (stroke (width 0.1) (type solid)) (layer "F.Fab"))
     (fp_circle (center 0 0) (end 1 0)
       (stroke (width 0.1) (type solid)) (fill none) (layer "F.Fab"))
-    (pad "1" smd roundrect (at -2.1 0 270) (size 0.8 2) (layers "F.Cu" "F.Paste" "F.Mask") (roundrect_rratio 0.25)
+    (pad "1" smd rect (at -3.1 -1.85 270) (size 1.8 1.1) (layers "F.Cu" "F.Paste" "F.Mask")
+      (net 2 "GND") (pinfunction "1") (pintype "passive"))
+    (pad "1" smd rect (at 3.1 -1.85 270) (size 1.8 1.1) (layers "F.Cu" "F.Paste" "F.Mask")
       (net 2 "GND") (pinfunction "1") (pintype "passive"))
-    (pad "2" smd roundrect (at 2.1 0 270) (size 0.8 2) (layers "F.Cu" "F.Paste" "F.Mask") (roundrect_rratio 0.25)
+    (pad "2" smd rect (at -3.1 1.85 270) (size 1.8 1.1) (layers "F.Cu" "F.Paste" "F.Mask")
       (net 4 "NRST") (pinfunction "2") (pintype "passive"))
-    (model "${KICAD6_3DMODEL_DIR}/Button_Switch_SMD.3dshapes/SW_Push_SPST_NO_Alps_SKRK.wrl"
+    (pad "2" smd rect (at 3.1 1.85 270) (size 1.8 1.1) (layers "F.Cu" "F.Paste" "F.Mask")
+      (net 4 "NRST") (pinfunction "2") (pintype "passive"))
+    (zone (net 0) (net_name "") (layer "F.Cu") (hatch full 0.508)
+      (connect_pads (clearance 0))
+      (min_thickness 0.254) (filled_areas_thickness no)
+      (keepout (tracks not_allowed) (vias not_allowed) (pads not_allowed) (copperpour not_allowed) (footprints not_allowed))
+      (fill (thermal_gap 0.508) (thermal_bridge_width 0.508))
+      (polygon
+        (pts
+          (xy 108.45625 96.0125)
+          (xy 108.45625 99.0125)
+          (xy 105.85625 99.0125)
+          (xy 105.85625 96.0125)
+        )
+      )
+    )
+    (zone (net 0) (net_name "") (layer "F.Cu") (hatch full 0.508)
+      (connect_pads (clearance 0))
+      (min_thickness 0.254) (filled_areas_thickness no)
+      (keepout (tracks not_allowed) (vias not_allowed) (pads not_allowed) (copperpour not_allowed) (footprints not_allowed))
+      (fill (thermal_gap 0.508) (thermal_bridge_width 0.508))
+      (polygon
+        (pts
+          (xy 108.45625 101.0125)
+          (xy 108.45625 104.0125)
+          (xy 105.85625 104.0125)
+          (xy 105.85625 101.0125)
+        )
+      )
+    )
+    (model "${KICAD6_3DMODEL_DIR}/Button_Switch_SMD.3dshapes/SW_SPST_SKQG_WithStem.wrl"
       (offset (xyz 0 0 0))
       (scale (xyz 1 1 1))
@@
   )
   (footprint "Capacitor_SMD:C_0805_2012Metric" (layer "B.Cu")
-    (at 106.3625 80.9625 -90)
+    (at 107.95 80.9625 -90)
     (descr "Capacitor SMD 0805 (2012 Metric), square (rectangular) end terminal, IPC_7351 nominal, (Body size source: IPC-SM-782 page 76, https://www.pcb-3d.com/wordpress/wp-content/uploads/ipc-sm-782a_amendment_1_and_2.pdf, https://docs.google.com/spreadsheets/d/1BsfQQcO9C6DZCsRaXUlFlo91Tg2WpOkGARC1WS5S8t0/edit?usp=sharing), generated with kicad-footprint-generator")
     (tags "capacitor")
@@
   )
   (footprint "Connector_USB:USB_C_Receptacle_HRO_TYPE-C-31-M-12" (layer "B.Cu")
-    (at 107.15625 27.78125)
+    (at 107.15625 29.36875)
     (descr "USB Type-C receptacle for USB 2.0 and PD, http://www.krhro.com/uploads/soft/180320/1-1P320120243.pdf")
     (tags "usb usb-c 2.0 pd")
     (property "Sheetfile" "intfield77.kicad_sch")
     (property "Sheetname" "")
-    (property "ki_description" "USB Full-Featured Type-C Receptacle connector")
-    (property "ki_keywords" "usb universal serial bus type-C full-featured")
+    (property "ki_description" "USB 2.0-only Type-C Receptacle connector")
+    (property "ki_keywords" "usb universal serial bus type-C USB2.0")
     (attr smd)
     (fp_text reference "J1" (at 0 5.645) (layer "B.SilkS")

Commit message: First routing of the PCB except the matrices.
Parts:
- C10: moved to F.Cu
- R1, R2, R3: footprint Resistor_SMD:R_0815_2038Metric -> Resistor_SMD:R_0805_2012Metric
- U2: footprint Package_TO_SOT_SMD:SOT-23-6 -> marbastlib-various:SOT-23-6-routable
- moved U2 11.2 mm to (108.0, 36.7), turned to 180 degrees
- moved C9 9.95 mm to (120.7, 48.4), turned to 90 degrees
- moved C8 8.73 mm to (114.3, 49.4)
- moved C4 6.20 mm to (115.1, 58.7)
- moved C3 5.78 mm to (101.6, 63.5), turned to 90 degrees
- moved C10 5.61 mm to (108.0, 97.6)
- moved U3 5.08 mm to (117.5, 48.4)
- moved C6 4.49 mm to (107.2, 77.8), turned to 0 degrees
- moved C1 4.38 mm to (114.3, 77.0), turned to 0 degrees
- moved R1 4.05 mm to (111.9, 34.9), turned to 0 degrees
- moved R2 4.05 mm to (104.0, 34.9)
- moved SW1 4.05 mm to (108.0, 104.0)
- moved C2 3.55 mm to (114.3, 74.6), turned to 0 degrees
- moved D20 3.37 mm to (95.2, 61.9)
- moved R3 2.86 mm to (119.9, 70.6), turned to 0 degrees
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Routing:
- net ROW8: track 0.00 -> 252.1 mm
- net COL3: track 0.00 -> 205.1 mm
- net COL4: track 0.00 -> 200.9 mm
- net GND: track 0.00 -> 192.8 mm, vias 0 -> 9
- net COL6: track 0.00 -> 180.1 mm
- net COL9: track 0.00 -> 177.5 mm
- net COL7: track 0.00 -> 167.2 mm
- net COL5: track 0.00 -> 164.2 mm
- net COL8: track 0.00 -> 160.3 mm
- net +3.3V: track 0.00 -> 139.8 mm, vias 0 -> 5
- net COL0: track 0.00 -> 83.2 mm
- net COL2: track 0.00 -> 78.5 mm
- net COL1: track 0.00 -> 58.3 mm
- net BOOT: track 0.00 -> 54.5 mm, vias 0 -> 1
- net ROW1: track 0.00 -> 52.8 mm
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Other:
- outline, holes or cut-outs redrawn

Commit message: Routing the matrices, but I might redo the pin assignments again.
Routing:
- net ROW7: track 4.44 -> 352.0 mm
- net ROW5: track 3.18 -> 331.4 mm
- net ROW3: track 4.67 -> 324.1 mm
- net ROW4: track 3.97 -> 306.3 mm
- net ROW6: track 4.30 -> 306.2 mm
- net ROW0: track 4.10 -> 297.1 mm
- net ROW2: track 4.02 -> 284.5 mm
- net ROW1: track 52.8 -> 322.4 mm
- net COL0: track 83.2 -> 170.8 mm
- net COL4: track 200.9 -> 277.7 mm
- net ROW8: track 252.1 -> 325.7 mm
- net COL1: track 58.3 -> 127.2 mm
- net ROW14: track 34.2 -> 85.5 mm
- net COL2: track 78.5 -> 126.1 mm
- net ROW13: track 42.3 -> 74.9 mm
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
Commit message: Reassigned pins and complete routing.
Parts:
- C10: moved to B.Cu
- moved C10 13.9 mm to (111.1, 84.1), turned to -90 degrees
- moved R3 2.51 mm to (119.1, 73.0), turned to -90 degrees
- moved D20 2.38 mm to (97.6, 61.9)
Connections:
- U1 pad 10: ROW3 -> COL5
- U1 pad 11: ROW4 -> COL4
- U1 pad 12: ROW5 -> COL3
- U1 pad 13: ROW6 -> ROW4
- U1 pad 14: ROW7 -> ROW5
- U1 pad 15: ROW8 -> ROW6
- U1 pad 16: unconnected-(U1-PA6-Pad16) -> ROW7
- U1 pad 17: unconnected-(U1-PA7-Pad17) -> ROW8
- U1 pad 18: ROW14 -> ROW12
- U1 pad 2: ROW0 -> COL8
- U1 pad 20: ROW12 -> ROW14
- U1 pad 21: ROW11 -> ROW10
- U1 pad 22: ROW10 -> ROW11
- U1 pad 3: ROW1 -> COL7
- U1 pad 39: COL9 -> ROW0
- U1 pad 4: ROW2 -> COL6
- U1 pad 40: COL8 -> ROW1
- U1 pad 41: COL7 -> ROW2
- U1 pad 42: COL6 -> ROW3
- U1 pad 43: COL5 -> COL9
- U1 pad 45: COL4 -> unconnected-(U1-PB8-Pad45)
- U1 pad 46: COL3 -> unconnected-(U1-PB9-Pad46)
Routing:
- net COL9: track 193.9 -> 448.5 mm
- net COL8: track 176.7 -> 397.8 mm
- net COL7: track 183.6 -> 366.9 mm
- net COL6: track 196.3 -> 342.0 mm
- net COL5: track 179.9 -> 304.2 mm
- net ROW14: track 85.5 -> 162.8 mm
- net ROW13: track 74.9 -> 141.9 mm
- net ROW12: track 56.4 -> 121.9 mm
- net ROW10: track 67.3 -> 128.9 mm
- net ROW11: track 48.4 -> 85.1 mm
- net ROW3: track 324.1 -> 287.8 mm
- net COL3: track 224.7 -> 254.8 mm
- net COL4: track 277.7 -> 303.0 mm
- net ROW0: track 297.1 -> 274.7 mm
- net ROW2: track 284.5 -> 264.1 mm
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
Commit message: Changed the silkscreen for the MX footprints.
Parts:
- MX1, MX10, MX11, MX12, MX13, MX14, MX15, MX16, MX18, MX19, MX2, MX20, MX22, MX23, MX24, MX25, MX26, MX27, MX28, MX29, MX3, MX30, MX31, MX32, MX33, MX35, MX36, MX37, MX39, MX4, MX40, MX41, MX42, MX43, MX44, MX45, MX46, MX47, MX48, MX49, MX5, MX51, MX52, MX53, MX55, MX56, MX57, MX58, MX59, MX6, MX60, MX61, MX62, MX63, MX64, MX65, MX66, MX67, MX69, MX7, MX75, MX76, MX77, MX8, MX9: footprint MX_Only:MXOnly-1U-NoLED -> local:MXOnly-1U-NoLED
- MX17, MX54, MX68: footprint MX_Only:MXOnly-2U-NoLED -> local:MXOnly-2U-NoLED
- MX21, MX34: footprint MX_Only:MXOnly-1.5U-NoLED -> local:MXOnly-1.5U-NoLED
- MX38: footprint MX_Only:MXOnly-1.75U-NoLED -> local:MXOnly-1.75U-NoLED
- MX50: footprint MX_Only:MXOnly-2.25U-NoLED -> local:MXOnly-2.25U-NoLED
- MX70, MX71, MX73, MX74: footprint MX_Only:MXOnly-1.25U-NoLED -> local:MXOnly-1.25U-NoLED
- MX72: footprint MX_Only:MXOnly-7U-NoLED -> local:MXOnly-7U-NoLED
